File: hardware/PCB_EU/MCU.kicad_sch (KiCad schematic)
At the start: 17 parts, among them J201 UART 3V3, SW201 RESET, SW202 BOOT, U201 AP63203WU-7, U202 ESP32-WROOM-32E-N4

Commit message: Port SS8PH10, ZL201-10G and terminal block changes from nikolajevs/ai PR #94
Apply the 20-file diff of nikolajevs/ai PR #94 (commit 63c79ad, merged as
7fa9410) on top of the 390374e import. Igors approved all three steps from
the 2026-10-23 shop price review (BOM 84.67 -> 81.25 EUR):

- D501/D601: SS5P10-M3/86A -> SS8PH10-M3/86A at Electrobase (same TO-277A
  land pattern, footprint and 3D model unchanged).
- J201: ZL2019-20 -> ZL201-10G at Salvats, cut 6 of 10 positions.
- DG306 bought 6 instead of 11, DG301R 1 instead of 2 (no spares).

hardware/PCB_EU now equals nikolajevs/ai at 7fa9410 except the two links
to PCB_V1 files in DESIGN.md and libraries/SOURCES.md that the import
rewrote. Reports in review/ are the ones saved by the full run of PR #94.

Co-Authored-By: Claude Sonnet 5.5 <noreply@anthropic.com>
Claude-Session: https://claude.ai/code/session_014SX1Gz36dYUdcXqtyGnqp6
Parts:
- J201: Design_note Cut 6 of purchased 20 header positions; 14 spare -> Cut 6 of purchased 10 header positions; 4 spare; MPN ZL2019-20 -> ZL201-10G
Changed lines of the file:
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@@
 (property "Footprint" "Connector_PinHeader_2.54mm:PinHeader_1x06_P2.54mm_Vertical" (at 106.68 185.42 0) (effects (font (size 1 1)) (hide yes)))
 (property "Datasheet" "" (at 106.68 185.42 0) (effects (font (size 1 1)) (hide yes)))
-(property "MPN" "ZL2019-20" (at 106.68 185.42 0) (effects (font (size 1 1)) (hide yes)))
-(property "Design_note" "Cut 6 of purchased 20 header positions; 14 spare" (at 106.68 185.42 0) (effects (font (size 1 1)) (hide yes)))
+(property "MPN" "ZL201-10G" (at 106.68 185.42 0) (effects (font (size 1 1)) (hide yes)))
+(property "Design_note" "Cut 6 of purchased 10 header positions; 4 spare" (at 106.68 185.42 0) (effects (font (size 1 1)) (hide yes)))
 (property "FootprintStatus" "PACKAGE ONLY - verify before PCB" (at 106.68 185.42 0) (effects (font (size 1 1)) (hide yes)))
 (pin "1")
