File: hardware/PCB_EU/LED2.kicad_sch (KiCad schematic)
At the start: 28 parts, among them J601 LED2 + / GND, J602 BAR2 + / GND, Q601 CSD19534KCS, U601 LM3429MH/NOPB

Commit message: Port SS8PH10, ZL201-10G and terminal block changes from nikolajevs/ai PR #94
Apply the 20-file diff of nikolajevs/ai PR #94 (commit 63c79ad, merged as
7fa9410) on top of the 390374e import. Igors approved all three steps from
the 2026-10-23 shop price review (BOM 84.67 -> 81.25 EUR):

- D501/D601: SS5P10-M3/86A -> SS8PH10-M3/86A at Electrobase (same TO-277A
  land pattern, footprint and 3D model unchanged).
- J201: ZL2019-20 -> ZL201-10G at Salvats, cut 6 of 10 positions.
- DG306 bought 6 instead of 11, DG301R 1 instead of 2 (no spares).

hardware/PCB_EU now equals nikolajevs/ai at 7fa9410 except the two links
to PCB_V1 files in DESIGN.md and libraries/SOURCES.md that the import
rewrote. Reports in review/ are the ones saved by the full run of PR #94.

Co-Authored-By: Claude Sonnet 5.5 <noreply@anthropic.com>
Claude-Session: https://claude.ai/code/session_014SX1Gz36dYUdcXqtyGnqp6
Parts:
- D601: value SS5P10 100V -> SS8PH10 100V; MPN SS5P10-M3/86A -> SS8PH10-M3/86A
Changed lines of the file:
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@@
 (symbol (lib_id "EU:D") (at 106.68 119.38 0) (unit 1) (in_bom yes) (on_board yes) (dnp no)
 (property "Reference" "D601" (at 106.68 113.74 0) (effects (font (size 1.15 1.15)) ))
-(property "Value" "SS5P10 100V" (at 106.68 125.02 0) (effects (font (size 0.98 0.98)) ))
+(property "Value" "SS8PH10 100V" (at 106.68 125.02 0) (effects (font (size 0.98 0.98)) ))
 (property "Footprint" "EU_Parts:Vishay_TO-277A_D_K1_A2" (at 106.68 119.38 0) (effects (font (size 1 1)) (hide yes)))
 (property "Datasheet" "" (at 106.68 119.38 0) (effects (font (size 1 1)) (hide yes)))
-(property "MPN" "SS5P10-M3/86A" (at 106.68 119.38 0) (effects (font (size 1 1)) (hide yes)))
+(property "MPN" "SS8PH10-M3/86A" (at 106.68 119.38 0) (effects (font (size 1 1)) (hide yes)))
 (property "Design_note" "" (at 106.68 119.38 0) (effects (font (size 1 1)) (hide yes)))
 (property "FootprintStatus" "PACKAGE ONLY - verify before PCB" (at 106.68 119.38 0) (effects (font (size 1 1)) (hide yes)))

Commit message: Replace dead-link KEMET 100n/100V with Samsung CL21B104KCFSFNE
The Electrobase card for C0805C104K1RACTU no longer opens. Use the
equivalent Samsung 100 nF / 100 V / X7R 0805 (0.12 EUR, live card) for
C511 and C611; BOM total is now 81.17 EUR.

Co-Authored-By: Claude Sonnet 5.5 <noreply@anthropic.com>
Parts:
- C611: MPN C0805C104K1RACTU -> CL21B104KCFSFNE
Changed lines of the file:
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@@
 (property "Footprint" "Capacitor_SMD:C_0805_2012Metric" (at 308.61 180.34 0) (effects (font (size 1 1)) (hide yes)))
 (property "Datasheet" "" (at 308.61 180.34 0) (effects (font (size 1 1)) (hide yes)))
-(property "MPN" "C0805C104K1RACTU" (at 308.61 180.34 0) (effects (font (size 1 1)) (hide yes)))
+(property "MPN" "CL21B104KCFSFNE" (at 308.61 180.34 0) (effects (font (size 1 1)) (hide yes)))
 (property "Design_note" "" (at 308.61 180.34 0) (effects (font (size 1 1)) (hide yes)))
 (property "FootprintStatus" "PACKAGE ONLY - verify before PCB" (at 308.61 180.34 0) (effects (font (size 1 1)) (hide yes)))
