File: hardware/PCB_EU/PCB_EU.kicad_pcb (KiCad board)
At the start: 4 copper layers, 100 x 100 mm, 201 parts, among them J101 24 V IN, J201 UART 3V3, J301 MEM2061 SPI, J401 SHT4x XH2.54-4P-90, J403 FLOAT / GND, J411 FAN1 2510-4P, J421 FAN2 2510-4P, J501 LED1 + / GND, J601 LED2 + / GND, J602 BAR2 + / GND, J701 PTC + / RETURN, J702 PUMP + / RETURN, Q102 FDB5800, Q411 FAN1 AO3422, Q421 FAN2 AO3422, Q501 TK22E10N1, Q601 CSD19534KCS, Q701 BC847B-DIO, Q702 BC857B, Q703 FDB5800, Q704 AO3422, SW201 RESET, SW202 BOOT, U101 L7987 3A, U102 INA226, U201 AP63203WU-7, U202 ESP32-WROOM-32E-N4, U301 MCP7940N-I/SN, U401 USBLC6-2SC6, U402 USBLC6-2SC6, U501 LM3429MH/NOPB, U601 LM3429MH/NOPB, U802 LM2903D-ST, Y301 32.768k CL7p

Commit message: Port SS8PH10, ZL201-10G and terminal block changes from nikolajevs/ai PR #94
Apply the 20-file diff of nikolajevs/ai PR #94 (commit 63c79ad, merged as
7fa9410) on top of the 390374e import. Igors approved all three steps from
the 2026-10-23 shop price review (BOM 84.67 -> 81.25 EUR):

- D501/D601: SS5P10-M3/86A -> SS8PH10-M3/86A at Electrobase (same TO-277A
  land pattern, footprint and 3D model unchanged).
- J201: ZL2019-20 -> ZL201-10G at Salvats, cut 6 of 10 positions.
- DG306 bought 6 instead of 11, DG301R 1 instead of 2 (no spares).

hardware/PCB_EU now equals nikolajevs/ai at 7fa9410 except the two links
to PCB_V1 files in DESIGN.md and libraries/SOURCES.md that the import
rewrote. Reports in review/ are the ones saved by the full run of PR #94.

Co-Authored-By: Claude Sonnet 5.5 <noreply@anthropic.com>
Claude-Session: https://claude.ai/code/session_014SX1Gz36dYUdcXqtyGnqp6
Parts:
- D501, D601: value SS5P10 100V -> SS8PH10 100V
Changed lines of the file:
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@@
 			)
 		)
-		(property "MPN" "ZL2019-20"
+		(property "MPN" "ZL201-10G"
 			(at 0 0 0)
 			(layer "F.SilkS")
@@
 			)
 		)
-		(property "Design_note" "Cut 6 of purchased 20 header positions; 14 spare"
+		(property "Design_note" "Cut 6 of purchased 10 header positions; 4 spare"
 			(at 0 0 0)
 			(layer "F.SilkS")
@@
 			)
 		)
-		(property "Value" "SS5P10 100V"
+		(property "Value" "SS8PH10 100V"
 			(at 0 4.5 90)
 			(layer "F.Fab")
@@
 			)
 		)
-		(property "MPN" "SS5P10-M3/86A"
+		(property "MPN" "SS8PH10-M3/86A"
 			(at 0 0 270)
 			(layer "F.SilkS")
@@
 			)
 		)
-		(property "Value" "SS5P10 100V"
+		(property "Value" "SS8PH10 100V"
 			(at 0 4.5 90)
 			(layer "F.Fab")
@@
 			)
 		)
-		(property "MPN" "SS5P10-M3/86A"
+		(property "MPN" "SS8PH10-M3/86A"
 			(at 0 0 270)
 			(layer "F.SilkS")
