File: hardware/PCB_EU_LITE/MCU.kicad_sch (KiCad schematic)
At the start: 23 parts, among them J201 UART 3V3, SW201 RESET, SW202 BOOT, U201 ST1S10PHR, U202 ESP32-WROOM-32E-N4

Commit message: Add RGB status LED to EU-LITE
Common-anode 5 mm RGB LED on +12V, three BC847B low-side switches driven from
GPIO4/16/17 (about 4.9/4.4/4.4 mA per channel, dark during reset). New
Status sheet, 56 script checks (5 more), 5 more mutation cases. The LED is in
neither the stock nor the catalogue snapshot: its BOM line has no price (the
estimate is stated separately). Docs carry a proposed status colour table; the
firmware is not changed.

Co-Authored-By: Claude <noreply@anthropic.com>
Claude-Session: https://claude.ai/code/session_013vgne5bRQcg5JyL7FL8xv5
Parts:
- U202: Design_note Antenna keepout and GND pad 39 mandatory; pins 6/7 (GPIO34/35, former tachometers) only pulled up -> Antenna keepout and GND pad 39 mandatory; pins 6/7 (GPIO34/35, former tachometers) only pulled up; pins 26/27/28 (GPIO4/16/17) drive the RGB status LED
Connections:
- net LED_R_GPIO: now reaches U202.26 (GPIO4)
- net LED_G_GPIO: now reaches U202.27 (GPIO16)
- net LED_B_GPIO: now reaches U202.28 (GPIO17)
- no-connect marks 16 -> 13
Changed lines of the file:
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@@
 (property "MPN" "ESP32-WROOM-32E-N4" (at 284.48 68.58 0) (effects (font (size 1 1)) (hide yes)))
 (property "Source" "buy" (at 284.48 68.58 0) (effects (font (size 1 1)) (hide yes)))
-(property "Design_note" "Antenna keepout and GND pad 39 mandatory; pins 6/7 (GPIO34/35, former tachometers) only pulled up" (at 284.48 68.58 0) (effects (font (size 1 1)) (hide yes)))
+(property "Design_note" "Antenna keepout and GND pad 39 mandatory; pins 6/7 (GPIO34/35, former tachometers) only pulled up; pins 26/27/28 (GPIO4/16/17) drive the RGB status LED" (at 284.48 68.58 0) (effects (font (size 1 1)) (hide yes)))
 (property "FootprintStatus" "DRAWING CHECKED in EU-0.1/cheap-version - physical fit pending" (at 284.48 68.58 0) (effects (font (size 1 1)) (hide yes)))
 (pin "1")
@@
 (global_label "SD_SCK_GPIO" (shape bidirectional) (at 312.42 64.77 0) (effects (font (size 0.9 0.9)) (justify left)) (property "Intersheetrefs" "${INTERSHEET_REFS}" (at 312.42 64.77 0) (effects (font (size 1 1)) (hide yes))))
 (no_connect (at 307.34 67.31))
-(no_connect (at 307.34 69.85))
-(no_connect (at 307.34 72.39))
-(no_connect (at 307.34 74.93))
+(wire (pts (xy 307.34 69.85) (xy 312.42 69.85)) (stroke (width 0) (type default)))
+(global_label "LED_B_GPIO" (shape bidirectional) (at 312.42 69.85 0) (effects (font (size 0.9 0.9)) (justify left)) (property "Intersheetrefs" "${INTERSHEET_REFS}" (at 312.42 69.85 0) (effects (font (size 1 1)) (hide yes))))
+(wire (pts (xy 307.34 72.39) (xy 312.42 72.39)) (stroke (width 0) (type default)))
+(global_label "LED_G_GPIO" (shape bidirectional) (at 312.42 72.39 0) (effects (font (size 0.9 0.9)) (justify left)) (property "Intersheetrefs" "${INTERSHEET_REFS}" (at 312.42 72.39 0) (effects (font (size 1 1)) (hide yes))))
+(wire (pts (xy 307.34 74.93) (xy 312.42 74.93)) (stroke (width 0) (type default)))
+(global_label "LED_R_GPIO" (shape bidirectional) (at 312.42 74.93 0) (effects (font (size 0.9 0.9)) (justify left)) (property "Intersheetrefs" "${INTERSHEET_REFS}" (at 312.42 74.93 0) (effects (font (size 1 1)) (hide yes))))
 (wire (pts (xy 307.34 77.47) (xy 312.42 77.47)) (stroke (width 0) (type default)))
 (global_label "ESP_BOOT" (shape bidirectional) (at 312.42 77.47 0) (effects (font (size 0.9 0.9)) (justify left)) (property "Intersheetrefs" "${INTERSHEET_REFS}" (at 312.42 77.47 0) (effects (font (size 1 1)) (hide yes))))
