File: hardware/PCB_EU_LITE/InputPower.kicad_sch (KiCad schematic)
At the start: 17 parts, among them J101 24 V IN, Q102 IRL2505, U102 INA238

Commit message: Fix EU-LITE footprint library resolution, verify ERC clean
fp-lib-table did not register a "Package_SO" library, so INA238's
custom VSSOP-10 footprint failed to resolve. Aliasing Package_SO to
PCB_EU's copy would have shadowed the stock exposed-pad SOIC-8
footprint that ST1S14/ST1S10 need from KiCad's bundled library.
Instead, move the two project-custom footprints (VSSOP-10 for INA238,
plain SOIC-8 for the MCP7940N RTC) into EU-LITE's own LITE_Parts
library with their 3D models, update generate.py accordingly, and
regenerate. Schematic and BOM are unchanged.

ERC (KiCad CLI 10.0.5): 0 violations. verify.py, check_schematics.py
and test_verify.py re-run clean.

Co-Authored-By: Claude Sonnet 5 <noreply@anthropic.com>
Parts:
- U102: footprint Package_SO:VSSOP-10_3x3mm_P0.5mm -> LITE_Parts:VSSOP-10_3x3mm_P0.5mm
Changed lines of the file:
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@@
 (property "Reference" "U102" (at 240.03 64.21 0) (effects (font (size 1.15 1.15)) ))
 (property "Value" "INA238" (at 240.03 85.65 0) (effects (font (size 0.98 0.98)) ))
-(property "Footprint" "Package_SO:VSSOP-10_3x3mm_P0.5mm" (at 240.03 74.93 0) (effects (font (size 1 1)) (hide yes)))
+(property "Footprint" "LITE_Parts:VSSOP-10_3x3mm_P0.5mm" (at 240.03 74.93 0) (effects (font (size 1 1)) (hide yes)))
 (property "Datasheet" "https://www.ti.com/lit/ds/symlink/ina238.pdf" (at 240.03 74.93 0) (effects (font (size 1 1)) (hide yes)))
 (property "MPN" "INA238AIDGSR" (at 240.03 74.93 0) (effects (font (size 1 1)) (hide yes)))
