File: hardware/PCB_EU_LITE/Peripherals.kicad_sch (KiCad schematic)
At the start: 18 parts, among them J301 MEM2061 SPI, U301 MCP7940N, Y301 32.768k CL7p

Commit message: Fix EU-LITE footprint library resolution, verify ERC clean
fp-lib-table did not register a "Package_SO" library, so INA238's
custom VSSOP-10 footprint failed to resolve. Aliasing Package_SO to
PCB_EU's copy would have shadowed the stock exposed-pad SOIC-8
footprint that ST1S14/ST1S10 need from KiCad's bundled library.
Instead, move the two project-custom footprints (VSSOP-10 for INA238,
plain SOIC-8 for the MCP7940N RTC) into EU-LITE's own LITE_Parts
library with their 3D models, update generate.py accordingly, and
regenerate. Schematic and BOM are unchanged.

ERC (KiCad CLI 10.0.5): 0 violations. verify.py, check_schematics.py
and test_verify.py re-run clean.

Co-Authored-By: Claude Sonnet 5 <noreply@anthropic.com>
Parts:
- U301: footprint Package_SO:SOIC-8_3.9x4.9mm_P1.27mm -> LITE_Parts:SOIC-8_3.9x4.9mm_P1.27mm
Changed lines of the file:
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@@
 (property "Reference" "U301" (at 74.93 50.24 0) (effects (font (size 1.15 1.15)) ))
 (property "Value" "MCP7940N" (at 74.93 69.14 0) (effects (font (size 0.98 0.98)) ))
-(property "Footprint" "Package_SO:SOIC-8_3.9x4.9mm_P1.27mm" (at 74.93 59.69 0) (effects (font (size 1 1)) (hide yes)))
+(property "Footprint" "LITE_Parts:SOIC-8_3.9x4.9mm_P1.27mm" (at 74.93 59.69 0) (effects (font (size 1 1)) (hide yes)))
 (property "Datasheet" "https://ww1.microchip.com/downloads/aemDocuments/documents/MPD/ProductDocuments/DataSheets/MCP7940N-Battery-Backed-I2C-RTCC-with-SRAM-20005010J.pdf" (at 74.93 59.69 0) (effects (font (size 1 1)) (hide yes)))
 (property "MPN" "MCP7940N-I/SN" (at 74.93 59.69 0) (effects (font (size 1 1)) (hide yes)))
