File: hardware/PCB_EU_LITE/Peripherals.kicad_sch (KiCad schematic)
At the start: 18 parts, among them J301 MEM2061 SPI, U301 MCP7940N, Y301 32.768k CL7p

Commit message: Move and route LITE RTC cluster near battery
Parts:
- BT301: footprint EU_Mechanical:Battery_COMF_BC-2001 -> LITE_Mechanical:Battery_COMF_BC-2001
Changed lines of the file:
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@@
 (property "Reference" "BT301" (at 308.61 113.74 0) (effects (font (size 1.15 1.15)) ))
 (property "Value" "CR2032 + BC-2001" (at 308.61 125.02 0) (effects (font (size 0.98 0.98)) ))
-(property "Footprint" "EU_Mechanical:Battery_COMF_BC-2001" (at 308.61 119.38 0) (effects (font (size 1 1)) (hide yes)))
+(property "Footprint" "LITE_Mechanical:Battery_COMF_BC-2001" (at 308.61 119.38 0) (effects (font (size 1 1)) (hide yes)))
 (property "Datasheet" "" (at 308.61 119.38 0) (effects (font (size 1 1)) (hide yes)))
 (property "MPN" "BC-2001" (at 308.61 119.38 0) (effects (font (size 1 1)) (hide yes)))
