File: hardware/PCB_EU_LITE/Status.kicad_sch (KiCad schematic)
At the start: 13 parts, among them Q901 BC847B (R), Q902 BC847B (G), Q903 BC847B (B)

Commit message: Refine EU-LITE placement and select RGB LED
Parts:
- D901: value RGB 5mm CA -> OSTAPA57E2A; footprint LED_THT:LED_D5.0mm-4_RGB -> LITE_Parts:LED_OSTAPA57E2A_Formed_P2.54mm; Design_note Not in stock and not in the catalogue snapshot: buy a 5 mm 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 -> Electrobase EB1854986288, owner quote 2026-10-25: EUR 0.85 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; MPN RGB-5MM-CA -> OSTAPA57E2A
Connections:
- net +12V: now also D901.3 (A); no longer D901.2 (A)
- net LED_B_K: now also D901.2 (B_K); no longer D901.4 (B_K)
- net LED_G_K: now also D901.1 (G_K); no longer D901.3 (G_K)
- net LED_R_K: now also D901.4 (R_K); no longer D901.1 (R_K)
Other:
- note added: "D901: OptoSupply OSTAPA57E2A, diffused RGB, COMMON ANODE on +12V. Pins 1 G, 2 B, 3 A, 4 R. Form leads from 1.25 to 2.54 mm pitch; body raised 5 mm above PCB. Each channel: GPIO -> 4k7 -> BC847B base (100k to GND), collector -> 2k -> LED cathode. The 12 V supply makes the current independent of the Vf of the green and blue dies (a 3.3 V supply leaves only 0.1-0.3 V across a resistor for Vf 3.0-3.2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"
- note removed: "D901: 5 mm diffused RGB LED, COMMON ANODE (owner decision 24.10.2026), anode on +12V. Lead order assumed R, A, G, B (KiCad LED_RAGB): confirm on the purchased part. Each channel: GPIO -> 4k7 -> BC847B base (100k to GND), collector -> 2k -> LED cathode. The 12 V supply makes the current independent of the Vf of the green and blue dies (a 3.3 V supply leaves only 0.1-0.3 V across a resistor for Vf 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"
Changed lines of the file:
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@@
 (kicad_sch (version 20260306) (generator "eeschema") (generator_version "10.0") (paper "A3") (title_block (title "08 | RGB status LED") (date "2026-10-24") (rev "EU-LITE-0.1") (company "GrowBox | EU-LITE from stock") (comment 1 "SCHEMATIC DRAFT | no PCB / manufacturing release"))
 (text "08 | RGB status LED" (at 12.7 12.7 0) (effects (font (size 2 2)) (justify left top)))
-(text "D901: 5 mm diffused RGB LED, COMMON ANODE (owner decision 24.10.2026), anode on +12V. Lead order assumed R, A, G, B (KiCad LED_RAGB): confirm on the purchased part.\nEach channel: GPIO -> 4k7 -> BC847B base (100k to GND), collector -> 2k -> LED cathode. The 12 V supply makes the current independent of the Vf of the green and blue dies\n(a 3.3 V supply leaves only 0.1-0.3 V across a resistor for Vf 3.0-3.2 V). ~4.9 mA red, ~4.4 mA green/blue; resistor 49 mW; 100k keeps the LED dark during reset.\nGPIO4 = red, GPIO16 = green, GPIO17 = blue (module pins 26/27/28; no strapping function, free on WROOM-32E-N4). Drive with LEDC PWM; HIGH = channel on.\nThe 12 V rail is off below ~14 V input, so the indicator is dark exactly when the ESP32 is not running." (at 12.7 251 0) (effects (font (size 1.02 1.02)) (justify left top)))
+(text "D901: OptoSupply OSTAPA57E2A, diffused RGB, COMMON ANODE on +12V. Pins 1 G, 2 B, 3 A, 4 R. Form leads from 1.25 to 2.54 mm pitch; body raised 5 mm above PCB.\nEach channel: GPIO -> 4k7 -> BC847B base (100k to GND), collector -> 2k -> LED cathode. The 12 V supply makes the current independent of the Vf of the green and blue dies\n(a 3.3 V supply leaves only 0.1-0.3 V across a resistor for Vf 3.0-3.2 V). ~4.9 mA red, ~4.4 mA green/blue; resistor 49 mW; 100k keeps the LED dark during reset.\nGPIO4 = red, GPIO16 = green, GPIO17 = blue (module pins 26/27/28; no strapping function, free on WROOM-32E-N4). Drive with LEDC PWM; HIGH = channel on.\nThe 12 V rail is off below ~14 V input, so the indicator is dark exactly when the ESP32 is not running." (at 12.7 251 0) (effects (font (size 1.02 1.02)) (justify left top)))
 (symbol (lib_id "EU_LITE:LED_RGB_CA") (at 119.38 69.85 0) (unit 1) (in_bom yes) (on_board yes) (dnp no)
 (property "Reference" "D901" (at 119.38 61.67 0) (effects (font (size 1.15 1.15)) ))
-(property "Value" "RGB 5mm CA" (at 119.38 78.03 0) (effects (font (size 0.98 0.98)) ))
-(property "Footprint" "LED_THT:LED_D5.0mm-4_RGB" (at 119.38 69.85 0) (effects (font (size 1 1)) (hide yes)))
-(property "Datasheet" "" (at 119.38 69.85 0) (effects (font (size 1 1)) (hide yes)))
-(property "MPN" "RGB-5MM-CA" (at 119.38 69.85 0) (effects (font (size 1 1)) (hide yes)))
+(property "Value" "OSTAPA57E2A" (at 119.38 78.03 0) (effects (font (size 0.98 0.98)) ))
+(property "Footprint" "LITE_Parts:LED_OSTAPA57E2A_Formed_P2.54mm" (at 119.38 69.85 0) (effects (font (size 1 1)) (hide yes)))
+(property "Datasheet" "https://www.optosupply.com/uppic/2020811188683.pdf" (at 119.38 69.85 0) (effects (font (size 1 1)) (hide yes)))
+(property "MPN" "OSTAPA57E2A" (at 119.38 69.85 0) (effects (font (size 1 1)) (hide yes)))
 (property "Source" "buy" (at 119.38 69.85 0) (effects (font (size 1 1)) (hide yes)))
-(property "Design_note" "Not in stock and not in the catalogue snapshot: buy a 5 mm diffused common-anode RGB LED (20 mA/channel max); check lead order and the color Vf (red ~2.0 V, green/blue ~3.0-3.3 V)" (at 119.38 69.85 0) (effects (font (size 1 1)) (hide yes)))
+(property "Design_note" "Electrobase EB1854986288, owner quote 2026-10-25: EUR 0.85 incl. VAT. Manufacturer Ver.a.1.1: flat top, pins G/B/A/R; formed-lead footprint, 1.0 mm holes, 1.8 mm pads. Check formed fit before soldering." (at 119.38 69.85 0) (effects (font (size 1 1)) (hide yes)))
 (property "FootprintStatus" "PACKAGE ONLY - verify before PCB" (at 119.38 69.85 0) (effects (font (size 1 1)) (hide yes)))
-(pin "2")
-(pin "1")
 (pin "3")
 (pin "4")
+(pin "1")
+(pin "2")
 (instances (project "PCB_EU_LITE" (path "/6650c329-4f4f-5b7a-a019-ee8e8f2772e1/7d73c2bc-1773-50f3-89a5-3aba4ffcc101" (reference "D901") (unit 1)))) )
 (wire (pts (xy 106.68 67.31) (xy 101.6 67.31)) (stroke (width 0) (type default)))
