File: hardware/PCB_EU_LITE/Interfaces.kicad_sch (KiCad schematic)
At the start: 18 parts, among them J401 SHT4x XH2.54-4P-90, J403 FLOAT / GND, J411 FAN1 2510-4P, J421 FAN2 2510-4P, Q411 FAN1 AO3422, Q421 FAN2 AO3422, U401 USBLC6-2SC6

Commit message: Move EU-LITE connectors to edges and add right-angle fan headers
Parts:
- J411: value FAN1 2510-4P -> FAN1 2510-4P 90deg; footprint Connector_Molex:Molex_KK-254_AE-6410-04A_1x04_P2.54mm_Vertical -> LITE_Parts:KF2510_1x04_P2.54mm_RightAngle; Design_note 4-pin PC fan pinout: 1 GND, 2 +12 V, 3 tach (NC), 4 PWM. KF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 -> Right-angle 2510-4AW footprint; stock KF2510/KF2540 variant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
- J421: value FAN2 2510-4P -> FAN2 2510-4P 90deg; footprint Connector_Molex:Molex_KK-254_AE-6410-04A_1x04_P2.54mm_Vertical -> LITE_Parts:KF2510_1x04_P2.54mm_RightAngle; Design_note 4-pin PC fan pinout: 1 GND, 2 +12 V, 3 tach (NC), 4 PWM. KF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 -> Right-angle 2510-4AW footprint; stock KF2510/KF2540 variant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
Changed lines of the file:
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@@
 (symbol (lib_id "EU_LITE:J4") (at 241.3 165.1 0) (unit 1) (in_bom yes) (on_board yes) (dnp no)
 (property "Reference" "J411" (at 241.3 155.65 0) (effects (font (size 1.15 1.15)) ))
-(property "Value" "FAN1 2510-4P" (at 241.3 174.55 0) (effects (font (size 0.98 0.98)) ))
-(property "Footprint" "Connector_Molex:Molex_KK-254_AE-6410-04A_1x04_P2.54mm_Vertical" (at 241.3 165.1 0) (effects (font (size 1 1)) (hide yes)))
+(property "Value" "FAN1 2510-4P 90deg" (at 241.3 174.55 0) (effects (font (size 0.98 0.98)) ))
+(property "Footprint" "LITE_Parts:KF2510_1x04_P2.54mm_RightAngle" (at 241.3 165.1 0) (effects (font (size 1 1)) (hide yes)))
 (property "Datasheet" "" (at 241.3 165.1 0) (effects (font (size 1 1)) (hide yes)))
 (property "MPN" "KF2510 / KF2540 4P" (at 241.3 165.1 0) (effects (font (size 1 1)) (hide yes)))
 (property "Source" "stock:87" (at 241.3 165.1 0) (effects (font (size 1 1)) (hide yes)))
-(property "Design_note" "4-pin PC fan pinout: 1 GND, 2 +12 V, 3 tach (NC), 4 PWM. KF2510 matches Molex KK-254; confirm against the part" (at 241.3 165.1 0) (effects (font (size 1 1)) (hide yes)))
+(property "Design_note" "Right-angle 2510-4AW footprint; stock KF2510/KF2540 variant needs physical confirmation. Pinout unchanged: 1 GND, 2 +12 V, 3 tach (NC), 4 PWM. Reference envelope: LHE A2543-WR04; check latch and pin 1 on actual part" (at 241.3 165.1 0) (effects (font (size 1 1)) (hide yes)))
 (property "FootprintStatus" "PACKAGE ONLY - verify before PCB" (at 241.3 165.1 0) (effects (font (size 1 1)) (hide yes)))
 (pin "1")
@@
 (symbol (lib_id "EU_LITE:J4") (at 45.72 185.42 0) (unit 1) (in_bom yes) (on_board yes) (dnp no)
 (property "Reference" "J421" (at 45.72 175.97 0) (effects (font (size 1.15 1.15)) ))
-(property "Value" "FAN2 2510-4P" (at 45.72 194.87 0) (effects (font (size 0.98 0.98)) ))
-(property "Footprint" "Connector_Molex:Molex_KK-254_AE-6410-04A_1x04_P2.54mm_Vertical" (at 45.72 185.42 0) (effects (font (size 1 1)) (hide yes)))
+(property "Value" "FAN2 2510-4P 90deg" (at 45.72 194.87 0) (effects (font (size 0.98 0.98)) ))
+(property "Footprint" "LITE_Parts:KF2510_1x04_P2.54mm_RightAngle" (at 45.72 185.42 0) (effects (font (size 1 1)) (hide yes)))
 (property "Datasheet" "" (at 45.72 185.42 0) (effects (font (size 1 1)) (hide yes)))
 (property "MPN" "KF2510 / KF2540 4P" (at 45.72 185.42 0) (effects (font (size 1 1)) (hide yes)))
 (property "Source" "stock:87" (at 45.72 185.42 0) (effects (font (size 1 1)) (hide yes)))
-(property "Design_note" "4-pin PC fan pinout: 1 GND, 2 +12 V, 3 tach (NC), 4 PWM. KF2510 matches Molex KK-254; confirm against the part" (at 45.72 185.42 0) (effects (font (size 1 1)) (hide yes)))
+(property "Design_note" "Right-angle 2510-4AW footprint; stock KF2510/KF2540 variant needs physical confirmation. Pinout unchanged: 1 GND, 2 +12 V, 3 tach (NC), 4 PWM. Reference envelope: LHE A2543-WR04; check latch and pin 1 on actual part" (at 45.72 185.42 0) (effects (font (size 1 1)) (hide yes)))
 (property "FootprintStatus" "PACKAGE ONLY - verify before PCB" (at 45.72 185.42 0) (effects (font (size 1 1)) (hide yes)))
 (pin "1")
