File: hardware/PCB_EU_LITE/LED.kicad_sch (KiCad schematic)
At the start: 38 parts, among them J501 LED + / GND, Q501 BSC146N10LS5, U501 LM3429MH/NOPB

Commit message: Finish EU-LITE LED routing and parallel outputs
Parts:
- added J502: LED 2 + / GND, TerminalBlock_Phoenix:TerminalBlock_Phoenix_MKDS-1,5-2_1x02_P5.00mm_Horizontal, symbol EU_LITE:J2
- added J503: LED 3 + / GND, TerminalBlock_Phoenix:TerminalBlock_Phoenix_MKDS-1,5-2_1x02_P5.00mm_Horizontal, symbol EU_LITE:J2
- Q501: Design_note Infineon OptiMOS 5 logic level: S1-S3, G4, D5-8. Stock: 2 p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 -> Infineon OptiMOS 5 logic level: S1-S3, G4, D5-8. One of two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
- R505: value 6k2 1% -> 4k7 1%; Design_note (none) -> With R506=620R: 5.32k total, ~1.55 A / 75 W-class at 48 V s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; MPN SMD1206-6K2-1% -> SMD1206 4K7 1%
- R506: value 1k2 1% -> 620R 1%; MPN CRCW12061K20FKTABC -> CRCW1206620RFKTABC
Connections:
- net GND: now also J502.2, J503.2
- net LED_POS: now also J502.1, J503.1
Other:
- note added: "J501/J502/J503 are parallel outputs AFTER R502: one 75 W-class LED channel, ~1.55 A TOTAL at ~48 V (1.235 V x 1k / (5.32k x 0.15 R)). LM3429 VIN senses the actual 24 V input. RCT is fed from SW through 56k + 6k2, CT 1 nF C0G: same as EU-0.1 LED1 (frequency unchanged). L501: stock Feryster DTMSS-27/0.047/15-V, 47 uH, 15 A, standing toroid ~35 mm high. Model peak <=4.36 A at 21.6 V, 90% efficiency,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"
- note removed: "One channel replaces the two of EU-0.1 (owner decision 24.10.2026): panel ~1.117 A nominal (1.24 V x 1k / (7.4k x 0.15 R)). A second load in parallel shares this current. LM3429 VIN senses the actual 24 V input. RCT is fed from SW through 56k + 6k2, CT 1 nF C0G: same as EU-0.1 LED1 (frequency unchanged). L501: stock Feryster DTMSS-27/0.047/15-V, 47 uH, 15 A, standing toroid ~35 mm high (cheap-ver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"
